File: projects/ohmify-overdrive/ohmify-overdrive.kicad_sch (KiCad schematic)
At the start: 18 parts, among them J1 InputJack, J2 OutputJack, U1 LM358

Commit message: Fixed 3DPT symbol for the overdrive
Connections:
- net INPUT: now also SW1.7; no longer SW1.8
- net OUTPUT: now also SW1.1; no longer SW1.2
- net at J1.T: now also SW1.8; no longer SW1.7
- net at J2.T: now also SW1.2; no longer SW1.1
Other:
- moved on the sheet: D3, R6, SW1B
Changed lines of the file:
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@@
   )
   (no_connect (at 72.39 82.55))
-  (no_connect (at 149.86 156.21))
+  (no_connect (at 158.369 154.94))
   (wire (pts (xy 40.64 146.05) (xy 40.64 151.13))
     (stroke (width 0) (type default))
@@
     (stroke (width 0) (type default))
   )
-  (wire (pts (xy 116.84 153.67) (xy 119.38 153.67))
+  (wire (pts (xy 135.509 149.86) (xy 138.049 149.86))
     (stroke (width 0) (type default))
   )
@@
     (stroke (width 0) (type default))
   )
-  (wire (pts (xy 127 153.67) (xy 129.54 153.67))
+  (wire (pts (xy 145.669 149.86) (xy 148.209 149.86))
     (stroke (width 0) (type default))
   )
@@
     (stroke (width 0) (type default))
   )
-  (wire (pts (xy 116.84 151.13) (xy 116.84 153.67))
+  (wire (pts (xy 135.509 147.32) (xy 135.509 149.86))
     (stroke (width 0) (type default))
   )
@@
     (stroke (width 0) (type default))
   )
-  (wire (pts (xy 153.67 151.13) (xy 149.86 151.13))
+  (wire (pts (xy 170.18 152.4) (xy 168.529 152.4))
     (stroke (width 0) (type default))
   )
@@
     (stroke (width 0) (type default))
   )
-  (wire (pts (xy 137.16 153.67) (xy 139.7 153.67))
+  (wire (pts (xy 155.829 149.86) (xy 158.369 149.86))
     (stroke (width 0) (type default))
   )
@@
     (stroke (width 0) (type default))
   )
-  (wire (pts (xy 153.67 154.94) (xy 153.67 151.13))
+  (wire (pts (xy 170.18 153.035) (xy 170.18 152.4))
     (stroke (width 0) (type default))
   )
@@
     )
   )
-  (symbol (lib_id "Device:LED") (at 133.35 153.67 180) (unit 1)
-    (in_bom yes) (on_board yes) (dnp no)
-    (property "Reference" "D3" (at 133.35 148.59 0)
-      (effects (font (size 1.27 1.27)))
-    )
-    (property "Value" "LED" (at 133.35 151.13 0)
-      (effects (font (size 1.27 1.27)))
-    )
-    (property "Footprint" "LED_THT:LED_D5.0mm" (at 133.35 153.67 0)
-      (effects (font (size 1.27 1.27)) hide)
-    )
-    (property "Datasheet" "~" (at 133.35 153.67 0)
+  (symbol (lib_id "Device:LED") (at 152.019 149.86 180) (unit 1)
+    (in_bom yes) (on_board yes) (dnp no)
+    (property "Reference" "D3" (at 152.019 144.78 0)
+      (effects (font (size 1.27 1.27)))
+    )
+    (property "Value" "LED" (at 152.019 147.32 0)
+      (effects (font (size 1.27 1.27)))
+    )
+    (property "Footprint" "LED_THT:LED_D5.0mm" (at 152.019 149.86 0)
+      (effects (font (size 1.27 1.27)) hide)
+    )
+    (property "Datasheet" "~" (at 152.019 149.86 0)
       (effects (font (size 1.27 1.27)) hide)
     )
@@
     )
   )
-  (symbol (lib_id "power:+9V") (at 116.84 151.13 0) (unit 1)
-    (in_bom yes) (on_board yes) (dnp no)
-    (property "Reference" "#PWR07" (at 116.84 154.94 0)
-      (effects (font (size 1.27 1.27)) hide)
-    )
-    (property "Value" "+9V" (at 116.84 147.32 0)
-      (effects (font (size 1.27 1.27)))
-    )
-    (property "Footprint" "" (at 116.84 151.13 0)
-      (effects (font (size 1.27 1.27)) hide)
-    )
-    (property "Datasheet" "" (at 116.84 151.13 0)
+  (symbol (lib_id "power:+9V") (at 135.509 147.32 0) (unit 1)
+    (in_bom yes) (on_board yes) (dnp no)
+    (property "Reference" "#PWR07" (at 135.509 151.13 0)
+      (effects (font (size 1.27 1.27)) hide)
+    )
+    (property "Value" "+9V" (at 135.509 143.51 0)
+      (effects (font (size 1.27 1.27)))
+    )
+    (property "Footprint" "" (at 135.509 147.32 0)
+      (effects (font (size 1.27 1.27)) hide)
+    )
+    (property "Datasheet" "" (at 135.509 147.32 0)
       (effects (font (size 1.27 1.27)) hide)
     )
@@
     )
   )
-  (symbol (lib_id "power:GND") (at 153.67 154.94 0) (unit 1)
-    (in_bom yes) (on_board yes) (dnp no)
-    (property "Reference" "#PWR08" (at 153.67 161.29 0)
-      (effects (font (size 1.27 1.27)) hide)
-    )
-    (property "Value" "GND" (at 153.67 158.75 0)
-      (effects (font (size 1.27 1.27)))
-    )
-    (property "Footprint" "" (at 153.67 154.94 0)
-      (effects (font (size 1.27 1.27)) hide)
-    )
-    (property "Datasheet" "" (at 153.67 154.94 0)
+  (symbol (lib_id "power:GND") (at 170.18 153.035 0) (unit 1)
+    (in_bom yes) (on_board yes) (dnp no)
+    (property "Reference" "#PWR08" (at 170.18 159.385 0)
+      (effects (font (size 1.27 1.27)) hide)
+    )
+    (property "Value" "GND" (at 170.18 156.845 0)
+      (effects (font (size 1.27 1.27)))
+    )
+    (property "Footprint" "" (at 170.18 153.035 0)
+      (effects (font (size 1.27 1.27)) hide)
+    )
+    (property "Datasheet" "" (at 170.18 153.035 0)
       (effects (font (size 1.27 1.27)) hide)
     )
@@
     )
   )
-  (symbol (lib_id "ohmify-switches:Switch_3PDT") (at 129.54 134.62 0) (unit 3)
+  (symbol (lib_name "Switch_3PDT_1") (lib_id "ohmify-switches:Switch_3PDT") (at 129.54 134.62 0) (unit 3)
     (in_bom yes) (on_board yes) (dnp no)
     (property "Reference" "SW1" (at 132.08 129.54 0)
@@
     )
   )
-  (symbol (lib_id "ohmify-switches:Switch_3PDT") (at 142.24 153.67 0) (unit 2)
-    (in_bom yes) (on_board yes) (dnp no) (fields_autoplaced)
-    (property "Reference" "SW1" (at 144.78 148.59 0)
-      (effects (font (size 1.27 1.27)))
-    )
-    (property "Value" "~" (at 142.24 153.67 0)
-      (effects (font (size 1.27 1.27)))
-    )
-    (property "Footprint" "Ohmify_Switches:Switch_3PDT" (at 142.24 153.67 0)
-      (effects (font (size 1.27 1.27)) hide)
-    )
-    (property "Datasheet" "" (at 142.24 153.67 0)
+  (symbol (lib_id "ohmify-switches:Switch_3PDT") (at 165.989 152.4 0) (mirror y) (unit 2)
+    (in_bom yes) (on_board yes) (dnp no)
+    (property "Reference" "SW1" (at 163.449 147.32 0)
+      (effects (font (size 1.27 1.27)))
+    )
+    (property "Value" "~" (at 165.989 152.4 0)
+      (effects (font (size 1.27 1.27)))
+    )
+    (property "Footprint" "Ohmify_Switches:Switch_3PDT" (at 165.989 152.4 0)
+      (effects (font (size 1.27 1.27)) hide)
+    )
+    (property "Datasheet" "" (at 165.989 152.4 0)
       (effects (font (size 1.27 1.27)) hide)
     )
@@
     )
   )
-  (symbol (lib_id "Device:R") (at 123.19 153.67 270) (unit 1)
-    (in_bom yes) (on_board yes) (dnp no)
-    (property "Reference" "R6" (at 121.92 151.13 90)
-      (effects (font (size 1.27 1.27)) (justify left))
-    )
-    (property "Value" "10k" (at 121.92 153.67 90)
-      (effects (font (size 1.27 1.27)) (justify left))
-    )
-    (property "Footprint" "Resistor_THT:R_Axial_DIN0207_L6.3mm_D2.5mm_P7.62mm_Horizontal" (at 123.19 151.892 90)
-      (effects (font (size 1.27 1.27)) hide)
-    )
-    (property "Datasheet" "~" (at 123.19 153.67 0)
+  (symbol (lib_id "Device:R") (at 141.859 149.86 270) (unit 1)
+    (in_bom yes) (on_board yes) (dnp no)
+    (property "Reference" "R6" (at 140.589 147.32 90)
+      (effects (font (size 1.27 1.27)) (justify left))
+    )
+    (property "Value" "10k" (at 140.589 149.86 90)
+      (effects (font (size 1.27 1.27)) (justify left))
+    )
+    (property "Footprint" "Resistor_THT:R_Axial_DIN0207_L6.3mm_D2.5mm_P7.62mm_Horizontal" (at 141.859 148.082 90)
+      (effects (font (size 1.27 1.27)) hide)
+    )
+    (property "Datasheet" "~" (at 141.859 149.86 0)
       (effects (font (size 1.27 1.27)) hide)
     )
@@
     )
   )
-  (symbol (lib_id "ohmify-switches:Switch_3PDT") (at 170.18 134.62 0) (mirror y) (unit 1)
+  (symbol (lib_name "Switch_3PDT_2") (lib_id "ohmify-switches:Switch_3PDT") (at 170.18 134.62 0) (mirror y) (unit 1)
     (in_bom yes) (on_board yes) (dnp no)
     (property "Reference" "SW1" (at 167.64 129.54 0)
