File: projects/ohmify-synthcard/ohmify-synthcard.kicad_sch (KiCad schematic)
At the start: 10 parts, among them U1 NE555P, U2 NE555P

Commit message: Fixed synthcard, added new gerber files
Connections:
- net at U1.3 (Q), U2.2 (TR): no longer RV1.3
- net at C1.1, U1.2 (TR): now also R1.1, U1.6 (THR)
- net at R1.2, U1.7 (DIS): now also RV1.3
Other:
- moved on the sheet: C1
Changed lines of the file:
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@@
   (title_block
     (title "SynthCard")
-    (rev "v1.0")
+    (date "2024-02-10")
+    (rev "v1.1")
     (company "Ohmify")
   )
-  (junction (at 152.4 104.14) (diameter 0) (color 0 0 0 0)
-  )
   (junction (at 118.11 80.01) (diameter 0) (color 0 0 0 0)
   )
@@
   (junction (at 135.89 77.47) (diameter 0) (color 0 0 0 0)
   )
+  (junction (at 149.86 114.3) (diameter 0) (color 0 0 0 0)
+  )
   (junction (at 203.2 114.3) (diameter 0) (color 0 0 0 0)
   )
+  (junction (at 120.65 120.523) (diameter 0) (color 0 0 0 0)
+  )
   (junction (at 135.89 130.81) (diameter 0) (color 0 0 0 0)
+  )
+  (junction (at 152.4 109.22) (diameter 0) (color 0 0 0 0)
   )
   (junction (at 171.45 80.01) (diameter 0) (color 0 0 0 0)
@@
     (stroke (width 0) (type default))
   )
-  (wire (pts (xy 152.4 95.25) (xy 152.4 104.14))
-    (stroke (width 0) (type default))
-  )
   (wire (pts (xy 118.11 114.3) (xy 118.11 80.01))
     (stroke (width 0) (type default))
@@
     (stroke (width 0) (type default))
   )
-  (wire (pts (xy 120.65 118.11) (xy 120.65 104.14))
+  (wire (pts (xy 120.65 120.523) (xy 120.65 104.14))
+    (stroke (width 0) (type default))
+  )
+  (wire (pts (xy 120.65 121.793) (xy 120.65 120.523))
+    (stroke (width 0) (type default))
+  )
+  (wire (pts (xy 149.86 114.3) (xy 151.13 114.3))
     (stroke (width 0) (type default))
   )
@@
     (stroke (width 0) (type default))
   )
-  (wire (pts (xy 120.65 125.73) (xy 120.65 130.81))
+  (wire (pts (xy 120.65 129.413) (xy 120.65 130.81))
     (stroke (width 0) (type default))
   )
@@
     (stroke (width 0) (type default))
   )
-  (wire (pts (xy 148.59 114.3) (xy 151.13 114.3))
+  (wire (pts (xy 148.59 114.3) (xy 149.86 114.3))
     (stroke (width 0) (type default))
   )
@@
     (stroke (width 0) (type default))
   )
+  (wire (pts (xy 152.4 95.25) (xy 152.4 109.22))
+    (stroke (width 0) (type default))
+  )
   (wire (pts (xy 203.2 80.01) (xy 203.2 86.36))
     (stroke (width 0) (type default))
@@
     (stroke (width 0) (type default))
   )
-  (wire (pts (xy 148.59 109.22) (xy 161.29 109.22))
+  (wire (pts (xy 149.86 114.3) (xy 149.86 120.523))
+    (stroke (width 0) (type default))
+  )
+  (wire (pts (xy 148.59 109.22) (xy 152.4 109.22))
     (stroke (width 0) (type default))
   )
@@
     (stroke (width 0) (type default))
   )
+  (wire (pts (xy 149.86 120.523) (xy 120.65 120.523))
+    (stroke (width 0) (type default))
+  )
   (wire (pts (xy 171.45 80.01) (xy 186.69 80.01))
     (stroke (width 0) (type default))
@@
     (stroke (width 0) (type default))
   )
-  (wire (pts (xy 148.59 104.14) (xy 152.4 104.14))
+  (wire (pts (xy 148.59 104.14) (xy 173.99 104.14))
     (stroke (width 0) (type default))
   )
@@
     (stroke (width 0) (type default))
   )
+  (wire (pts (xy 152.4 109.22) (xy 161.29 109.22))
+    (stroke (width 0) (type default))
+  )
   (wire (pts (xy 152.4 86.36) (xy 152.4 87.63))
     (stroke (width 0) (type default))
@@
   )
   (wire (pts (xy 157.48 91.44) (xy 156.21 91.44))
-    (stroke (width 0) (type default))
-  )
-  (wire (pts (xy 152.4 104.14) (xy 173.99 104.14))
     (stroke (width 0) (type default))
   )
@@
     (pin "2")
     (instances
-      (project "SynthCard"
+      (project "ohmify-synthcard"
         (path "/ba5ae891-fc98-44d2-bcac-f784448702be"
           (reference "RV2") (unit 1)
@@
     (pin "1")
     (instances
-      (project "SynthCard"
+      (project "ohmify-synthcard"
         (path "/ba5ae891-fc98-44d2-bcac-f784448702be"
           (reference "#FLG01") (unit 1)
@@
     (pin "2")
     (instances
-      (project "SynthCard"
+      (project "ohmify-synthcard"
         (path "/ba5ae891-fc98-44d2-bcac-f784448702be"
           (reference "C2") (unit 1)
@@
     (pin "1")
     (instances
-      (project "SynthCard"
+      (project "ohmify-synthcard"
         (path "/ba5ae891-fc98-44d2-bcac-f784448702be"
           (reference "BT1") (unit 1)
@@
     (pin "4")
     (instances
-      (project "SynthCard"
+      (project "ohmify-synthcard"
         (path "/ba5ae891-fc98-44d2-bcac-f784448702be"
           (reference "U2") (unit 1)
@@
     (pin "2")
     (instances
-      (project "SynthCard"
+      (project "ohmify-synthcard"
         (path "/ba5ae891-fc98-44d2-bcac-f784448702be"
           (reference "RV1") (unit 1)
@@
     )
   )
-  (symbol (lib_id "Device:C") (at 120.65 121.92 0) (unit 1)
+  (symbol (lib_id "Device:C") (at 120.65 125.603 0) (unit 1)
     (in_bom yes) (on_board yes) (dnp no)
-    (property "Reference" "C1" (at 123.19 120.65 0)
-      (effects (font (size 1.27 1.27)) (justify left))
-    )
-    (property "Value" "10nF" (at 123.19 123.19 0)
-      (effects (font (size 1.27 1.27)) (justify left))
-    )
-    (property "Footprint" "Capacitor_THT:C_Rect_L7.0mm_W2.5mm_P5.00mm" (at 121.6152 125.73 0)
-      (effects (font (size 1.27 1.27)) hide)
-    )
-    (property "Datasheet" "~" (at 120.65 121.92 0)
-      (effects (font (size 1.27 1.27)) hide)
-    )
-    (pin "1")
-    (pin "2")
-    (instances
-      (project "SynthCard"
+    (property "Reference" "C1" (at 123.19 124.333 0)
+      (effects (font (size 1.27 1.27)) (justify left))
+    )
+    (property "Value" "10nF" (at 123.19 126.873 0)
+      (effects (font (size 1.27 1.27)) (justify left))
+    )
+    (property "Footprint" "Capacitor_THT:C_Rect_L7.0mm_W2.5mm_P5.00mm" (at 121.6152 129.413 0)
+      (effects (font (size 1.27 1.27)) hide)
+    )
+    (property "Datasheet" "~" (at 120.65 125.603 0)
+      (effects (font (size 1.27 1.27)) hide)
+    )
+    (pin "1")
+    (pin "2")
+    (instances
+      (project "ohmify-synthcard"
         (path "/ba5ae891-fc98-44d2-bcac-f784448702be"
           (reference "C1") (unit 1)
@@
     (pin "1")
     (instances
-      (project "SynthCard"
+      (project "ohmify-synthcard"
         (path "/ba5ae891-fc98-44d2-bcac-f784448702be"
           (reference "#PWR02") (unit 1)
@@
     (pin "2")
     (instances
-      (project "SynthCard"
+      (project "ohmify-synthcard"
         (path "/ba5ae891-fc98-44d2-bcac-f784448702be"
           (reference "R1") (unit 1)
@@
     (pin "1")
     (instances
-      (project "SynthCard"
+      (project "ohmify-synthcard"
         (path "/ba5ae891-fc98-44d2-bcac-f784448702be"
           (reference "#PWR01") (unit 1)
@@
     (pin "1")
     (instances
-      (project "SynthCard"
+      (project "ohmify-synthcard"
         (path "/ba5ae891-fc98-44d2-bcac-f784448702be"
           (reference "#FLG02") (unit 1)
@@
     (pin "4")
     (instances
-      (project "SynthCard"
+      (project "ohmify-synthcard"
         (path "/ba5ae891-fc98-44d2-bcac-f784448702be"
           (reference "U1") (unit 1)
@@
     (pin "2")
     (instances
-      (project "SynthCard"
+      (project "ohmify-synthcard"
         (path "/ba5ae891-fc98-44d2-bcac-f784448702be"
           (reference "C3") (unit 1)
@@
     (pin "1")
     (instances
-      (project "SynthCard"
+      (project "ohmify-synthcard"
         (path "/ba5ae891-fc98-44d2-bcac-f784448702be"
           (reference "LS1") (unit 1)

Commit message: Working v1.1 synthcard
Parts:
- C2: value 10nF -> 100nF
Other:
- moved on the sheet: C1, C2, C3, LS1, R1, RV1, RV2, U1, U2
